Commit message: managed to introduce the robot in gazebo

File: robot_bringup/urdf/robot_rviz.urdf.xacro (robot description, xacro)
@@ -32,7 +32,13 @@
             <origin rpy="${pi/2} 0 0" xyz="0 0 0"/>
             <geometry>
-              <mesh filename="file://$(find robot_bringup)/robot_mesh/base_link.dae"/>
-              <!-- <box size="0.3 0.3 0.3"/> -->
+              <!-- <mesh filename="file://$(find robot_bringup)/robot_mesh/base_link.dae"/>  -->
+              <box size="0.3 0.3 0.3"/>
             </geometry>
+          </collision>
+          <inertial>
+            <mass value="50000"/>
+            <inertia ixx="0.4" ixy="0.0" ixz="0.0" iyy="0.4" iyz="0.0" izz="0.2"/>
+          </inertial>
+          <surface>
             <friction>
               <ode>
@@ -41,9 +47,5 @@
               </ode>
             </friction>
-          </collision>
-          <inertial>
-            <mass value="50000"/>
-            <inertia ixx="40" ixy="0.0" ixz="0.0" iyy="40" iyz="0.0" izz="20"/>
-          </inertial>
+            </surface>
             <selfCollide>false</selfCollide>
     </link >
@@ -55,13 +57,13 @@
         </geometry>
       </visual>
-      <collision>
+      <!-- <collision>
         <origin rpy="${pi/2} 0 ${pi/2}" xyz="0 0 0"/>
         <geometry>
           <mesh filename="file://$(find robot_bringup)/robot_mesh/link1.dae"/>
         </geometry>
-      </collision>
-      <inertial>
-        <mass value="1000"/>
-        <inertia ixx="40" ixy="0.0" ixz="0.0" iyy="40" iyz="0.0" izz="20"/>
+      </collision> -->
+      <inertial>
+        <mass value="1000"/>
+        <inertia ixx="0.4" ixy="0.0" ixz="0.0" iyy="0.4" iyz="0.0" izz="0.2"/>
       </inertial>
       <selfCollide>false</selfCollide>
@@ -74,13 +76,13 @@
         </geometry>
       </visual>
-      <collision>
+      <!-- <collision>
         <origin rpy="-${pi/2} 0 ${pi}" xyz="0 0 0"/>
         <geometry>
           <mesh filename="file://$(find robot_bringup)/robot_mesh/link2.dae"/>
         </geometry>
-      </collision>
-      <inertial>
-        <mass value="1000"/>
-        <inertia ixx="40" ixy="0.0" ixz="0.0" iyy="40" iyz="0.0" izz="20"/>
+      </collision> -->
+      <inertial>
+        <mass value="1000"/>
+        <inertia ixx="0.4" ixy="0.0" ixz="0.0" iyy="0.4" iyz="0.0" izz="0.2"/>
       </inertial>
       <selfCollide>false</selfCollide>
@@ -93,13 +95,13 @@
         </geometry>
       </visual>
-      <collision>
+      <!-- <collision>
         <origin rpy="${pi/2} 0 ${pi}" xyz="0 0 0"/>
         <geometry>
           <mesh filename="file://$(find robot_bringup)/robot_mesh/link3.dae"/>
         </geometry>
-      </collision>
-      <inertial>
-        <mass value="1000"/>
-        <inertia ixx="40" ixy="0.0" ixz="0.0" iyy="40" iyz="0.0" izz="20"/>
+      </collision> -->
+      <inertial>
+        <mass value="1000"/>
+        <inertia ixx="0.4" ixy="0.0" ixz="0.0" iyy="0.4" iyz="0.0" izz="0.2"/>
       </inertial>
       <selfCollide>false</selfCollide>
@@ -108,5 +110,5 @@
       <inertial>
         <mass value="10"/>
-        <inertia ixx="40" ixy="0.0" ixz="0.0" iyy="40" iyz="0.0" izz="20"/>
+        <inertia ixx="0.0004" ixy="0.0" ixz="0.0" iyy="0.0004" iyz="0.0" izz="0.0002"/>
       </inertial>
       <selfCollide>false</selfCollide>
@@ -119,13 +121,13 @@
         </geometry>
       </visual>
-      <collision>
+      <!-- <collision>
         <origin rpy="${pi} ${pi/2} 0" xyz="0 0 0"/>
         <geometry>
           <mesh filename="file://$(find robot_bringup)/robot_mesh/link4.dae"/>
         </geometry>
-      </collision>
-      <inertial>
-        <mass value="1000"/>
-        <inertia ixx="40" ixy="0.0" ixz="0.0" iyy="40" iyz="0.0" izz="20"/>
+      </collision> -->
+      <inertial>
+        <mass value="1000"/>
+        <inertia ixx="0.4" ixy="0.0" ixz="0.0" iyy="0.4" iyz="0.0" izz="0.2"/>
       </inertial>
       <selfCollide>false</selfCollide>
@@ -134,9 +136,9 @@
       <inertial>
         <mass value="10"/>
-        <inertia ixx="40" ixy="0.0" ixz="0.0" iyy="40" iyz="0.0" izz="20"/>
-      </inertial>
-      <selfCollide>false</selfCollide>
-    </link >
-    <!-- <link name="link4_1" >
+        <inertia ixx="0.004" ixy="0.0" ixz="0.0" iyy="0.004" iyz="0.0" izz="0.002"/>
+      </inertial>
+      <selfCollide>false</selfCollide>
+    </link >
+    <link name="link4_1" >
       <visual>
         <origin rpy="${pi} ${pi/2} 0.261" xyz="0 0 0"/>
@@ -198,5 +200,4 @@
       </inertial>
     </link >
-   -->
     <!-- Joints Declaration -->
     <joint name="dummy_joint" type="fixed">
@@ -211,5 +212,4 @@
       <axis xyz="0 0 1" />
       <origin xyz="0 0 0.2645" rpy="0 0 0" />
-      <dynamics damping="0.5" friction="0.0"/>
     </joint>
     <joint name="joint2" type="revolute">
@@ -219,5 +219,4 @@
       <axis xyz="0 0 1" />
       <origin xyz="0.21938 0.1675 0.332" rpy="${pi/2} 0 0" />
-      <dynamics damping="0.5" friction="0.0"/>
     </joint>
     <joint name="joint3" type="revolute">
@@ -227,5 +226,4 @@
       <axis xyz="0 0 1" />
       <origin xyz="0 1.100 0" rpy="0 0 0" />
-      <dynamics damping="0.5" friction="0.0"/>
     </joint>
     <joint name="joint4_artificial" type="continuous">
@@ -245,5 +243,4 @@
       <axis xyz="0 0 1" />
       <origin xyz="0 0 0" rpy="0 0 0" />
-      <dynamics damping="0.5" friction="0.0"/>
     </joint>
     <xacro:mimic_joint_plugin_gazebo name_prefix="joint4"
@@ -256,7 +253,6 @@
       <limit effort="1000.0" lower="${-360*pi/180}" upper="${360*pi/180}" velocity="${148*pi/180}"/>
       <origin xyz="0.1718 -0.18957 0" rpy="${pi/2} 0 0" />
-      <dynamics damping="0.5" friction="0.0"/>
-    </joint>
-    <!-- <joint name="joint4_1" type="continuous">
+    </joint>
+    <joint name="joint4_1" type="continuous">
       <mimic joint="joint2" multiplier="-1" offset="0" />
       <parent link="link1"/>
@@ -285,5 +281,5 @@
       <axis xyz="0 0 1" />
       <origin xyz="0 0 0" rpy="0 0 0" />
-    </joint> -->
+    </joint>
     <!-- Transmission -->
     <gazebo>
