Commit message: started adding meshes

File: robot_bringup/urdf/robot.urdf (robot description, URDF)
Before this commit: robot test_robot, 4 links, 3 joints
Links:
- removed link base
- added link base_link; visual mesh filename=file://$(find robot_bringup)/robot_mesh/base_link.dae
- link link1: geometry 
- link link2: geometry 
- link link3: geometry 
Joints:
- removed joint base_to_link1
- removed joint link1_to_link2
- removed joint link2_to_link3
- added joint joint1: type continuous, parent base_link, child link1, origin xyz=0 0 1 rpy=0 0 0, axis 0 0 1
- added joint joint2: type continuous, parent link1, child link2, origin xyz=1 0 0 rpy=0 0 0, axis 0 0 1
- added joint joint3: type prismatic, parent link2, child link3, origin xyz=1 0 0 rpy=0 1.57 0, limit lower=0.0 upper=0.548 effort=1000.0 velocity=0.5

Commit message: added meshes

File: robot_bringup/urdf/robot.urdf (robot description, URDF)
Before this commit: robot test_robot, 4 links, 3 joints
Links:
- link link1: geometry visual mesh filename=file://$(find robot_bringup)/robot_mesh/link1.dae
- link link2: geometry visual mesh filename=file://$(find robot_bringup)/robot_mesh/link2.dae
- link link3: geometry visual mesh filename=file://$(find robot_bringup)/robot_mesh/link3.dae
Joints:
- joint joint1: origin xyz=0 0 1 rpy=0 0 0 -> xyz=0 0 276 rpy=0 0 0
- joint joint2: origin xyz=1 0 0 rpy=0 0 0 -> xyz=247 200 335 rpy=1.57 0 0
- joint joint3: axis (none) -> 0 0 1; limit lower=0.0 upper=0.548 effort=1000.0 velocity=0.5 -> (none); origin xyz=1 0 0 rpy=0 1.57 0 -> xyz=1100 0 0 rpy=0 0 0; type prismatic -> continuous

Commit message: added meshes

File: robot_bringup/urdf/robot.urdf (robot description, URDF)
Before this commit: robot test_robot, 4 links, 3 joints
Joints:
- joint joint1: origin xyz=0 0 276 rpy=0 0 0 -> xyz=0 0 264.5 rpy=0 0 0
- joint joint2: origin xyz=247 200 335 rpy=1.57 0 0 -> xyz=247 168.02 332 rpy=1.57 0 0

Commit message: finished the robot model

File: robot_bringup/urdf/robot.urdf (robot description, URDF)
Before this commit: robot test_robot, 4 links, 3 joints
Links:
- added link link4; visual mesh filename=file://$(find robot_bringup)/robot_mesh/link4.dae
- added link link4_1; visual mesh filename=file://$(find robot_bringup)/robot_mesh/link4_1.dae
- added link link4_2; visual mesh filename=file://$(find robot_bringup)/robot_mesh/link4_2.dae
- added link link4_3; visual mesh filename=file://$(find robot_bringup)/robot_mesh/link4_3.dae
- added link link4_3_artificial
- added link link4_artificial
Joints:
- added joint joint4: type continuous, parent link4_artificial, child link4, origin xyz=0 0 0 rpy=0 0 0, axis 0 0 1, mimic joint=joint3 multiplier=-1 offset=0
- added joint joint4_1: type continuous, parent link1, child link4_1, origin xyz=-84.21 61.92 376.87 rpy=-1.57 0.02 0, axis 0 0 1, mimic joint=joint2 multiplier=-1 offset=0
- added joint joint4_2: type continuous, parent link4_1, child link4_2, origin xyz=10 -1100 -24.5 rpy=0 0 -0.15, axis 0 0 1, mimic joint=joint2 multiplier=1 offset=0
- added joint joint4_3: type continuous, parent link4_3_artificial, child link4_3, origin xyz=0 0 0 rpy=0 0 0, axis 0 0 1, mimic joint=joint3 multiplier=-1 offset=0
- added joint joint4_3_artificial: type continuous, parent link4_2, child link4_3_artificial, origin xyz=583.29 0 -70 rpy=0 0 0, axis 0 0 1, mimic joint=joint2 multiplier=-1 offset=0
- added joint joint4_artificial: type continuous, parent link3, child link4_artificial, origin xyz=972.83 0 102.5 rpy=0 0 0, axis 0 0 1, mimic joint=joint2 multiplier=-1 offset=0
- joint joint2: origin xyz=247 168.02 332 rpy=1.57 0 0 -> xyz=247 168.02 332 rpy=1.57 -1.57 0
- joint joint3: origin xyz=1100 0 0 rpy=0 0 0 -> xyz=1100 0 0 rpy=0 0 -1.57

Commit message: added robot to gazebo

File: robot_bringup/urdf/robot.urdf (robot description, URDF)
Before this commit: robot test_robot, 10 links, 9 joints
Links:
- added link link5, mass 10
- link base_link: mass None -> 50000; geometry collision mesh filename=file://$(find robot_bringup)/robot_mesh/base_link.dae; visual mesh filename=file://$(find robot_bringup)/robot_mesh/base_link.dae
- link link1: mass None -> 1000; geometry collision mesh filename=file://$(find robot_bringup)/robot_mesh/link1.dae; visual mesh filename=file://$(find robot_bringup)/robot_mesh/link1.dae
- link link2: mass None -> 1000; geometry collision mesh filename=file://$(find robot_bringup)/robot_mesh/link2.dae; visual mesh filename=file://$(find robot_bringup)/robot_mesh/link2.dae
- link link3: mass None -> 1000; geometry collision mesh filename=file://$(find robot_bringup)/robot_mesh/link3.dae; visual mesh filename=file://$(find robot_bringup)/robot_mesh/link3.dae
- link link4: mass None -> 1000; geometry collision mesh filename=file://$(find robot_bringup)/robot_mesh/link4.dae; visual mesh filename=file://$(find robot_bringup)/robot_mesh/link4.dae
- link link4_1: mass None -> 1000; geometry collision mesh filename=file://$(find robot_bringup)/robot_mesh/link4_1.dae; visual mesh filename=file://$(find robot_bringup)/robot_mesh/link4_1.dae
- link link4_2: mass None -> 1000; geometry collision mesh filename=file://$(find robot_bringup)/robot_mesh/link4_2.dae; visual mesh filename=file://$(find robot_bringup)/robot_mesh/link4_2.dae
- link link4_3: mass None -> 1000; geometry collision mesh filename=file://$(find robot_bringup)/robot_mesh/link4_3.dae; visual mesh filename=file://$(find robot_bringup)/robot_mesh/link4_3.dae
- link link4_3_artificial: mass None -> 10
- link link4_artificial: mass None -> 10
Joints:
- added joint joint5: type continuous, parent link4, child link5, origin xyz=0.17227 -0.18953 0 rpy=1.57 0 0, axis 0 0 1
- joint joint1: origin xyz=0 0 264.5 rpy=0 0 0 -> xyz=0 0 0.2645 rpy=0 0 0
- joint joint2: origin xyz=247 168.02 332 rpy=1.57 -1.57 0 -> xyz=0.247 0.16802 0.332 rpy=1.57 0 0
- joint joint3: origin xyz=1100 0 0 rpy=0 0 -1.57 -> xyz=0 1.100 0 rpy=0 0 0
- joint joint4_1: origin xyz=-84.21 61.92 376.87 rpy=-1.57 0.02 0 -> xyz=-0.08421 0.06192 0.37687 rpy=-1.57 0.02 0
- joint joint4_2: origin xyz=10 -1100 -24.5 rpy=0 0 -0.15 -> xyz=0.010 -1.100 -0.0245 rpy=0 0 -0.15
- joint joint4_3_artificial: origin xyz=583.29 0 -70 rpy=0 0 0 -> xyz=0.58329 0 -0.070 rpy=0 0 0
- joint joint4_artificial: origin xyz=972.83 0 102.5 rpy=0 0 0 -> xyz=0.97283 0 0.1025 rpy=0 0 0

Commit message: added a function to get the last frame coordinates

File: robot_bringup/urdf/robot.urdf (robot description, URDF)
Before this commit: robot robot, 11 links, 10 joints
Links:
- link base_link: mass 50000 -> 10000
