Commit message: finalized gazebo but need to fix rviz mesh

File: robot_bringup/urdf/robot.urdf (robot description, URDF)
Before this commit: robot robot, 7 links, 6 joints
Links:
- link base_link: geometry visual mesh filename=file://$(find robot_bringup)/robot_mesh/base_link.dae
- link link1: mass 1000 -> None; geometry visual mesh filename=file://$(find robot_bringup)/robot_mesh/link1.dae
- link link2: mass 1000 -> None; geometry visual mesh filename=file://$(find robot_bringup)/robot_mesh/link2.dae
- link link3: mass 1000 -> None; geometry visual mesh filename=file://$(find robot_bringup)/robot_mesh/link3.dae
- link link4: mass 1000 -> None; geometry visual mesh filename=file://$(find robot_bringup)/robot_mesh/link4.dae
- link link4_artificial: mass 10 -> None
- link link5: mass 10 -> None
Joints:
- joint joint1: limit lower=0.0 upper=0.548 effort=1000.0 velocity=0.5 -> (none)
- joint joint2: limit lower=0.0 upper=0.548 effort=1000.0 velocity=0.5 -> (none)
- joint joint3: limit lower=0.0 upper=0.548 effort=1000.0 velocity=0.5 -> (none)
- joint joint4: limit lower=0.0 upper=0.548 effort=1000.0 velocity=0.5 -> (none)
- joint joint4_artificial: limit lower=0.0 upper=0.548 effort=1000.0 velocity=0.5 -> (none)
- joint joint5: limit lower=0.0 upper=0.548 effort=1000.0 velocity=0.5 -> (none)

File: robot_bringup/urdf/robot.urdf.xacro (robot description, xacro)
@@ -19,5 +19,5 @@
     </gazebo>
   </xacro:macro>
-    <xacro:property name="path" value="model://" />
+    <xacro:property name="path" value="model://robot_mesh" />
     <link name="dummy_link" >
     </link >
@@ -26,5 +26,5 @@
             <origin rpy="${pi/2} 0 0" xyz="0 0 0"/>
             <geometry>
-              <mesh filename="file://$(find robot_bringup)/robot_mesh/base_link.dae"/>
+              <mesh filename="${path}/base_link.dae"/>
             </geometry>
           </visual>
@@ -32,5 +32,5 @@
             <origin rpy="${pi/2} 0 0" xyz="0 0 0"/>
             <geometry>
-              <mesh filename="file://$(find robot_bringup)/robot_mesh/base_link.dae"/>
+              <mesh filename="${path}/base_link.dae"/>
               <!-- <box size="0.3 0.3 0.3"/> -->
             </geometry>
@@ -44,5 +44,5 @@
           <inertial>
             <mass value="50000"/>
-            <inertia ixx="40" ixy="0.0" ixz="0.0" iyy="40" iyz="0.0" izz="20"/>
+            <inertia ixx="750.000000" ixy="-0.000115" ixz="0.003024" iyy="1040.000000" iyz="-90.592690" izz="1040.000000"/>
           </inertial>
             <selfCollide>false</selfCollide>
@@ -52,5 +52,5 @@
         <origin rpy="${pi/2} 0 ${pi/2}" xyz="0 0 0"/>
         <geometry>
-          <mesh filename="file://$(find robot_bringup)/robot_mesh/link1.dae"/>
+          <mesh filename="${path}/link1.dae"/>
         </geometry>
       </visual>
@@ -58,5 +58,95 @@
         <origin rpy="${pi/2} 0 ${pi/2}" xyz="0 0 0"/>
         <geometry>
-          <mesh filename="file://$(find robot_bringup)/robot_mesh/link1.dae"/>
+          <mesh filename="${path}/link1.dae"/>
+        </geometry>
+      </collision>
+      <inertial>
+        <mass value="20000"/>
+        <inertia ixx="40" ixy="0.0" ixz="0.0" iyy="40" iyz="0.0" izz="40"/>
+      </inertial>
+      <selfCollide>false</selfCollide>
+    </link >
+    <link name="link2" >
+      <visual>
+        <origin rpy="-${pi/2} 0 ${pi}" xyz="0 0 0"/>
+        <geometry>
+          <mesh filename="${path}/link2.dae"/>
+        </geometry>
+      </visual>
+      <collision>
+        <origin rpy="-${pi/2} 0 ${pi}" xyz="0 0 0"/>
+        <geometry>
+          <mesh filename="${path}/link2.dae"/>
+        </geometry>
+      </collision>
+      <inertial>
+        <mass value="1000"/>
+        <inertia ixx="20" ixy="0.0" ixz="0.0" iyy="20" iyz="0.0" izz="20"/>
+      </inertial>
+      <selfCollide>false</selfCollide>
+    </link >
+    <link name="link3" >
+      <visual>
+        <origin rpy="${pi/2} 0 ${pi}" xyz="0 0 0"/>
+        <geometry>
+          <mesh filename="${path}/link3.dae"/>
+        </geometry>
+      </visual>
+      <collision>
+        <origin rpy="${pi/2} 0 ${pi}" xyz="0 0 0"/>
+        <geometry>
+          <mesh filename="${path}/link3.dae"/>
+        </geometry>
+      </collision>
+      <inertial>
+        <mass value="1000"/>
+        <inertia ixx="10" ixy="0.0" ixz="0.0" iyy="10" iyz="0.0" izz="10"/>
+      </inertial>
+      <selfCollide>false</selfCollide>
+    </link >
+    <link name="link4_artificial" >
+      <inertial>
+        <mass value="10"/>
+        <inertia ixx="0.001" ixy="0.0" ixz="0.0" iyy="0.001" iyz="0.0" izz="0.001"/>
+      </inertial>
+      <selfCollide>false</selfCollide>
+    </link >
+    <link name="link4" >
+      <visual>
+        <origin rpy="${pi} ${pi/2} 0" xyz="0 0 0"/>
+        <geometry>
+          <mesh filename="${path}/link4.dae"/>
+        </geometry>
+      </visual>
+      <collision>
+        <origin rpy="${pi} ${pi/2} 0" xyz="0 0 0"/>
+        <geometry>
+          <mesh filename="${path}/link4.dae"/>
+        </geometry>
+      </collision>
+      <inertial>
+        <mass value="1000"/>
+        <inertia ixx="5" ixy="0.0" ixz="0.0" iyy="5" iyz="0.0" izz="5"/>
+      </inertial>
+      <selfCollide>false</selfCollide>
+    </link >
+    <link name="link5" >
+      <inertial>
+        <mass value="1"/>
+        <inertia ixx="0.001" ixy="0.0" ixz="0.0" iyy="0.001" iyz="0.0" izz="0.001"/>
+      </inertial>
+      <selfCollide>false</selfCollide>
+    </link >
+    <!-- <link name="link4_1" >
+      <visual>
+        <origin rpy="${pi} ${pi/2} 0.261" xyz="0 0 0"/>
+        <geometry>
+          <mesh filename="${path}/link4_1.dae"/>
+        </geometry>
+      </visual>
+      <collision>
+        <origin rpy="${pi} ${pi/2} 0.261" xyz="0 0 0"/>
+        <geometry>
+          <mesh filename="${path}/link4_1.dae"/>
         </geometry>
       </collision>
@@ -65,17 +155,16 @@
         <inertia ixx="40" ixy="0.0" ixz="0.0" iyy="40" iyz="0.0" izz="20"/>
       </inertial>
-      <selfCollide>false</selfCollide>
-    </link >
-    <link name="link2" >
-      <visual>
-        <origin rpy="-${pi/2} 0 ${pi}" xyz="0 0 0"/>
-        <geometry>
-          <mesh filename="file://$(find robot_bringup)/robot_mesh/link2.dae"/>
-        </geometry>
-      </visual>
-      <collision>
-        <origin rpy="-${pi/2} 0 ${pi}" xyz="0 0 0"/>
-        <geometry>
-          <mesh filename="file://$(find robot_bringup)/robot_mesh/link2.dae"/>
+    </link >
+    <link name="link4_2" >
+      <visual>
+        <origin rpy="${pi} ${pi/2} ${pi/2}" xyz="0 0 0"/>
+        <geometry>
+          <mesh filename="${path}/link4_2.dae"/>
+        </geometry>
+      </visual>
+      <collision>
+        <origin rpy="${pi} ${pi/2} ${pi/2}" xyz="0 0 0"/>
+        <geometry>
+          <mesh filename="${path}/link4_2.dae"/>
         </geometry>
       </collision>
@@ -84,43 +173,22 @@
         <inertia ixx="40" ixy="0.0" ixz="0.0" iyy="40" iyz="0.0" izz="20"/>
       </inertial>
-      <selfCollide>false</selfCollide>
-    </link >
-    <link name="link3" >
-      <visual>
-        <origin rpy="${pi/2} 0 ${pi}" xyz="0 0 0"/>
-        <geometry>
-          <mesh filename="file://$(find robot_bringup)/robot_mesh/link3.dae"/>
-        </geometry>
-      </visual>
-      <collision>
-        <origin rpy="${pi/2} 0 ${pi}" xyz="0 0 0"/>
-        <geometry>
-          <mesh filename="file://$(find robot_bringup)/robot_mesh/link3.dae"/>
-        </geometry>
-      </collision>
-      <inertial>
-        <mass value="1000"/>
-        <inertia ixx="40" ixy="0.0" ixz="0.0" iyy="40" iyz="0.0" izz="20"/>
-      </inertial>
-      <selfCollide>false</selfCollide>
-    </link >
-    <link name="link4_artificial" >
+    </link >
+    <link name="link4_3_artificial" >
       <inertial>
         <mass value="10"/>
         <inertia ixx="40" ixy="0.0" ixz="0.0" iyy="40" iyz="0.0" izz="20"/>
       </inertial>
-      <selfCollide>false</selfCollide>
-    </link >
-    <link name="link4" >
-      <visual>
-        <origin rpy="${pi} ${pi/2} 0" xyz="0 0 0"/>
-        <geometry>
-          <mesh filename="file://$(find robot_bringup)/robot_mesh/link4.dae"/>
-        </geometry>
-      </visual>
-      <collision>
-        <origin rpy="${pi} ${pi/2} 0" xyz="0 0 0"/>
-        <geometry>
-          <mesh filename="file://$(find robot_bringup)/robot_mesh/link4.dae"/>
+    </link >
+    <link name="link4_3" >
+      <visual>
+        <origin rpy="0 0 0.12" xyz="0 0 0"/>
+        <geometry>
+          <mesh filename="${path}/link4_3.dae"/>
+        </geometry>
+      </visual>
+      <collision>
+        <origin rpy="0 0 0.12" xyz="0 0 0"/>
+        <geometry>
+          <mesh filename="${path}/link4_3.dae"/>
         </geometry>
       </collision>
@@ -129,74 +197,5 @@
         <inertia ixx="40" ixy="0.0" ixz="0.0" iyy="40" iyz="0.0" izz="20"/>
       </inertial>
-      <selfCollide>false</selfCollide>
-    </link >
-    <link name="link5" >
-      <inertial>
-        <mass value="10"/>
-        <inertia ixx="40" ixy="0.0" ixz="0.0" iyy="40" iyz="0.0" izz="20"/>
-      </inertial>
-      <selfCollide>false</selfCollide>
-    </link >
-    <!-- <link name="link4_1" >
-      <visual>
-        <origin rpy="${pi} ${pi/2} 0.261" xyz="0 0 0"/>
-        <geometry>
-          <mesh filename="file://$(find robot_bringup)/robot_mesh/link4_1.dae"/>
-        </geometry>
-      </visual>
-      <collision>
-        <origin rpy="${pi} ${pi/2} 0.261" xyz="0 0 0"/>
-        <geometry>
-          <mesh filename="file://$(find robot_bringup)/robot_mesh/link4_1.dae"/>
-        </geometry>
-      </collision>
-      <inertial>
-        <mass value="1000"/>
-        <inertia ixx="0.4" ixy="0.0" ixz="0.0" iyy="0.4" iyz="0.0" izz="0.2"/>
-      </inertial>
-    </link >
-    <link name="link4_2" >
-      <visual>
-        <origin rpy="${pi} ${pi/2} ${pi/2}" xyz="0 0 0"/>
-        <geometry>
-          <mesh filename="file://$(find robot_bringup)/robot_mesh/link4_2.dae"/>
-        </geometry>
-      </visual>
-      <collision>
-        <origin rpy="${pi} ${pi/2} ${pi/2}" xyz="0 0 0"/>
-        <geometry>
-          <mesh filename="file://$(find robot_bringup)/robot_mesh/link4_2.dae"/>
-        </geometry>
-      </collision>
-      <inertial>
-        <mass value="1000"/>
-        <inertia ixx="0.4" ixy="0.0" ixz="0.0" iyy="0.4" iyz="0.0" izz="0.2"/>
-      </inertial>
-    </link >
-    <link name="link4_3_artificial" >
-      <inertial>
-        <mass value="10"/>
-        <inertia ixx="0.4" ixy="0.0" ixz="0.0" iyy="0.4" iyz="0.0" izz="0.2"/>
-      </inertial>
-    </link >
-    <link name="link4_3" >
-      <visual>
-        <origin rpy="0 0 0.12" xyz="0 0 0"/>
-        <geometry>
-          <mesh filename="file://$(find robot_bringup)/robot_mesh/link4_3.dae"/>
-        </geometry>
-      </visual>
-      <collision>
-        <origin rpy="0 0 0.12" xyz="0 0 0"/>
-        <geometry>
-          <mesh filename="file://$(find robot_bringup)/robot_mesh/link4_3.dae"/>
-        </geometry>
-      </collision>
-      <inertial>
-        <mass value="1000"/>
-        <inertia ixx="0.4" ixy="0.0" ixz="0.0" iyy="0.4" iyz="0.0" izz="0.2"/>
-      </inertial>
-    </link >
-   -->
+    </link > -->
     <!-- Joints Declaration -->
     <joint name="dummy_joint" type="fixed">
@@ -208,5 +207,5 @@
       <parent link="base_link"/>
       <child link="link1"/>
-      <limit effort="100.0" lower="${-175*pi/180}" upper="${175*pi/180}" velocity="${60*pi/180}"/>
+      <limit effort="100000.0" lower="${-175*pi/180}" upper="${175*pi/180}" velocity="${60*pi/180}"/>
       <axis xyz="0 0 1" />
       <origin xyz="0 0 0.2645" rpy="0 0 0" />
@@ -216,5 +215,5 @@
       <parent link="link1"/>
       <child link="link2"/>
-      <limit effort="100.0" lower="${-25*pi/180}" upper="${80*pi/180}" velocity="${148*pi/180}"/>
+      <limit effort="1000000.0" lower="${-25*pi/180}" upper="${80*pi/180}" velocity="${148*pi/180}"/>
       <axis xyz="0 0 1" />
       <origin xyz="0.21938 0.1675 0.332" rpy="${pi/2} 0 0" />
@@ -224,5 +223,5 @@
       <parent link="link2"/>
       <child link="link3"/>
-      <limit effort="100.0" lower="${-25*pi/180}" upper="${80*pi/180}" velocity="${148*pi/180}"/>
+      <limit effort="1000000.0" lower="${-25*pi/180}" upper="${80*pi/180}" velocity="${148*pi/180}"/>
       <axis xyz="0 0 1" />
       <origin xyz="0 1.100 0" rpy="0 0 0" />
@@ -238,5 +237,5 @@
     <xacro:mimic_joint_plugin_gazebo name_prefix="joint4_artificial"
     parent_joint="joint2" mimic_joint="joint4_artificial"
-    has_pid="false" multiplier="-1.0" max_effort="10.0" />
+    has_pid="false" multiplier="-1.0" max_effort="10.0" robot_namespace="/robot" />
     <joint name="joint4" type="continuous">
       <mimic joint="joint3" multiplier="-1" offset="0" />
@@ -249,10 +248,10 @@
     <xacro:mimic_joint_plugin_gazebo name_prefix="joint4"
     parent_joint="joint3" mimic_joint="joint4"
-    has_pid="false" multiplier="-1.0" max_effort="10.0" />
+    has_pid="false" multiplier="-1.0" max_effort="10.0" robot_namespace="/robot" />
     <joint name="joint5" type="revolute">
       <parent link="link4"/>
       <child link="link5"/>
       <axis xyz="0 0 1" />
-      <limit effort="1000.0" lower="${-360*pi/180}" upper="${360*pi/180}" velocity="${148*pi/180}"/>
+      <limit effort="10.0" lower="${-360*pi/180}" upper="${360*pi/180}" velocity="${148*pi/180}"/>
       <origin xyz="0.1718 -0.18957 0" rpy="${pi/2} 0 0" />
       <dynamics damping="0.5" friction="0.0"/>
@@ -265,4 +264,7 @@
       <origin xyz="-0.08421 0.06192 0.37687" rpy="-${pi/2} 0.02 0" />
     </joint>
+    <xacro:mimic_joint_plugin_gazebo name_prefix="joint4"
+    parent_joint="joint2" mimic_joint="joint4_1"
+    has_pid="false" multiplier="-1.0" max_effort="10.0"  robot_namespace="/robot"/>
     <joint name="joint4_2" type="continuous">
       <mimic joint="joint2" multiplier="1" offset="0" />
@@ -272,6 +274,9 @@
       <origin xyz="0.010 -1.100 -0.0245" rpy="0 0 -0.15" />
     </joint>
+    <xacro:mimic_joint_plugin_gazebo name_prefix="joint4"
+    parent_joint="joint2" mimic_joint="joint4_2"
+    has_pid="false" multiplier="1.0" max_effort="10.0" robot_namespace="/robot" />
     <joint name="joint4_3_artificial" type="continuous">
-      <mimic joint="joint2" multiplier="-1" offset="0" />
+      <mimic joint="joint2" multiplier="-1" offset="0"  />
       <parent link="link4_2"/>
       <child link="link4_3_artificial"/>
@@ -279,4 +284,7 @@
       <origin xyz="0.58329 0 -0.070" rpy="0 0 0" />
     </joint>
+    <xacro:mimic_joint_plugin_gazebo name_prefix="joint4"
+    parent_joint="joint2" mimic_joint="joint4_3_artificial"
+    has_pid="false" multiplier="-1.0" max_effort="10.0" robot_namespace="/robot"/>
     <joint name="joint4_3" type="continuous">
       <mimic joint="joint3" multiplier="-1" offset="0" />
@@ -285,10 +293,13 @@
       <axis xyz="0 0 1" />
       <origin xyz="0 0 0" rpy="0 0 0" />
-    </joint> -->
+    </joint>
+    <xacro:mimic_joint_plugin_gazebo name_prefix="joint4"
+    parent_joint="joint3" mimic_joint="joint4_3"
+    has_pid="false" multiplier="-1.0" max_effort="10.0" robot_namespace="/robot"/> -->
     <!-- Transmission -->
+    <!-- Gazebo control plugin -->
     <gazebo>
       <plugin name="gazebo_ros_control" filename="libgazebo_ros_control.so">
         <robotNamespace>/robot</robotNamespace>
-        <robotSimType>gazebo_ros_control/DefaultRobotHWSim</robotSimType>
       </plugin>
     </gazebo>
@@ -297,8 +308,8 @@
       <actuator name="motor1">
         <mechanicalReduction>1</mechanicalReduction>
-        <hardwareInterface>hardware_interface/EffortJointInterface</hardwareInterface>
+        <hardwareInterface>hardware_interface/PositionJointInterface</hardwareInterface>
       </actuator>
       <joint name="joint1">
-        <hardwareInterface>hardware_interface/EffortJointInterface</hardwareInterface>
+        <hardwareInterface>hardware_interface/PositionJointInterface</hardwareInterface>
       </joint>
     </transmission>
@@ -307,8 +318,8 @@
       <actuator name="motor2">
         <mechanicalReduction>1</mechanicalReduction>
-        <hardwareInterface>hardware_interface/EffortJointInterface</hardwareInterface>
+        <hardwareInterface>hardware_interface/PositionJointInterface</hardwareInterface>
       </actuator>
       <joint name="joint2">
-        <hardwareInterface>hardware_interface/EffortJointInterface</hardwareInterface>
+        <hardwareInterface>hardware_interface/PositionJointInterface</hardwareInterface>
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
File: robot_bringup/urdf/robot_rviz.urdf.xacro (robot description, xacro)
@@ -19,4 +19,5 @@
     </gazebo>
   </xacro:macro>
+   <xacro:property name="path" value="/media/andre/Andre/robot_mesh" />
     <!-- <xacro:property name="pi" value="3.14" /> -->
     <link name="dummy_link" >
@@ -26,5 +27,5 @@
             <origin rpy="${pi/2} 0 0" xyz="0 0 0"/>
             <geometry>
-              <mesh filename="file://$(find robot_bringup)/robot_mesh/base_link.dae"/>
+              <mesh filename="${path}/base_link.dae"/>
             </geometry>
           </visual>
@@ -32,5 +33,5 @@
             <origin rpy="${pi/2} 0 0" xyz="0 0 0"/>
             <geometry>
-              <!-- <mesh filename="file://$(find robot_bringup)/robot_mesh/base_link.dae"/>  -->
+              <!-- <mesh filename="${path}/base_link.dae"/>  -->
               <box size="0.3 0.3 0.3"/>
             </geometry>
@@ -54,5 +55,5 @@
         <origin rpy="${pi/2} 0 ${pi/2}" xyz="0 0 0"/>
         <geometry>
-          <mesh filename="file://$(find robot_bringup)/robot_mesh/link1.dae"/>
+          <mesh filename="${path}/link1.dae"/>
         </geometry>
       </visual>
@@ -60,5 +61,5 @@
         <origin rpy="${pi/2} 0 ${pi/2}" xyz="0 0 0"/>
         <geometry>
-          <mesh filename="file://$(find robot_bringup)/robot_mesh/link1.dae"/>
+          <mesh filename="${path}/link1.dae"/>
         </geometry>
       </collision> -->
@@ -73,5 +74,5 @@
         <origin rpy="-${pi/2} 0 ${pi}" xyz="0 0 0"/>
         <geometry>
-          <mesh filename="file://$(find robot_bringup)/robot_mesh/link2.dae"/>
+          <mesh filename="${path}/link2.dae"/>
         </geometry>
       </visual>
@@ -79,5 +80,5 @@
         <origin rpy="-${pi/2} 0 ${pi}" xyz="0 0 0"/>
         <geometry>
-          <mesh filename="file://$(find robot_bringup)/robot_mesh/link2.dae"/>
+          <mesh filename="${path}/link2.dae"/>
         </geometry>
       </collision> -->
@@ -92,5 +93,5 @@
         <origin rpy="${pi/2} 0 ${pi}" xyz="0 0 0"/>
         <geometry>
-          <mesh filename="file://$(find robot_bringup)/robot_mesh/link3.dae"/>
+          <mesh filename="${path}/link3.dae"/>
         </geometry>
       </visual>
@@ -98,5 +99,5 @@
         <origin rpy="${pi/2} 0 ${pi}" xyz="0 0 0"/>
         <geometry>
-          <mesh filename="file://$(find robot_bringup)/robot_mesh/link3.dae"/>
+          <mesh filename="${path}/link3.dae"/>
         </geometry>
       </collision> -->
@@ -118,5 +119,5 @@
         <origin rpy="${pi} ${pi/2} 0" xyz="0 0 0"/>
         <geometry>
-          <mesh filename="file://$(find robot_bringup)/robot_mesh/link4.dae"/>
+          <mesh filename="${path}/link4.dae"/>
         </geometry>
       </visual>
@@ -124,5 +125,5 @@
         <origin rpy="${pi} ${pi/2} 0" xyz="0 0 0"/>
         <geometry>
-          <mesh filename="file://$(find robot_bringup)/robot_mesh/link4.dae"/>
+          <mesh filename="${path}/link4.dae"/>
         </geometry>
       </collision> -->
@@ -144,5 +145,5 @@
         <origin rpy="${pi} ${pi/2} 0.261" xyz="0 0 0"/>
         <geometry>
-          <mesh filename="file://$(find robot_bringup)/robot_mesh/link4_1.dae"/>
+          <mesh filename="${path}/link4_1.dae"/>
         </geometry>
       </visual>
@@ -150,5 +151,5 @@
         <origin rpy="${pi} ${pi/2} 0.261" xyz="0 0 0"/>
         <geometry>
-          <mesh filename="file://$(find robot_bringup)/robot_mesh/link4_1.dae"/>
+          <mesh filename="${path}/link4_1.dae"/>
         </geometry>
       </collision>
@@ -162,5 +163,5 @@
         <origin rpy="${pi} ${pi/2} ${pi/2}" xyz="0 0 0"/>
         <geometry>
-          <mesh filename="file://$(find robot_bringup)/robot_mesh/link4_2.dae"/>
+          <mesh filename="${path}/link4_2.dae"/>
         </geometry>
       </visual>
@@ -168,5 +169,5 @@
         <origin rpy="${pi} ${pi/2} ${pi/2}" xyz="0 0 0"/>
         <geometry>
-          <mesh filename="file://$(find robot_bringup)/robot_mesh/link4_2.dae"/>
+          <mesh filename="${path}/link4_2.dae"/>
         </geometry>
       </collision>
@@ -186,5 +187,5 @@
         <origin rpy="0 0 0.12" xyz="0 0 0"/>
         <geometry>
-          <mesh filename="file://$(find robot_bringup)/robot_mesh/link4_3.dae"/>
+          <mesh filename="${path}/link4_3.dae"/>
         </geometry>
       </visual>
@@ -192,5 +193,5 @@
         <origin rpy="0 0 0.12" xyz="0 0 0"/>
         <geometry>
-          <mesh filename="file://$(find robot_bringup)/robot_mesh/link4_3.dae"/>
+          <mesh filename="${path}/link4_3.dae"/>
         </geometry>
       </collision>
