Commit message: added direct kinematics

File: robot_bringup/urdf/robot.urdf.xacro (robot description, xacro)
@@ -1,6 +1,8 @@
-<robot name="robot">
+<?xml version="1.0"?>
+<robot xmlns:xacro="http://www.ros.org/wiki/xacro" name="robot">
+    <!-- <xacro:property name="pi" value="3.14" /> -->
     <link name="base_link" >
         <visual>
-            <origin rpy="1.57 0 0" xyz="0 0 0"/>
+            <origin rpy="${pi/2} 0 0" xyz="0 0 0"/>
             <geometry>
               <mesh filename="file://$(find robot_bringup)/robot_mesh/base_link.dae"/>
@@ -8,5 +10,5 @@
           </visual>
           <collision>
-            <origin rpy="1.57 0 0" xyz="0 0 0"/>
+            <origin rpy="${pi/2} 0 0" xyz="0 0 0"/>
             <geometry>
               <mesh filename="file://$(find robot_bringup)/robot_mesh/base_link.dae"/>
@@ -21,5 +23,5 @@
     <link name="link1">
       <visual>
-        <origin rpy="1.57 0 1.57" xyz="0 0 0"/>
+        <origin rpy="${pi/2} 0 ${pi/2}" xyz="0 0 0"/>
         <geometry>
           <mesh filename="file://$(find robot_bringup)/robot_mesh/link1.dae"/>
@@ -27,5 +29,5 @@
       </visual>
       <collision>
-        <origin rpy="1.57 0 1.57" xyz="0 0 0"/>
+        <origin rpy="${pi/2} 0 ${pi/2}" xyz="0 0 0"/>
         <geometry>
           <mesh filename="file://$(find robot_bringup)/robot_mesh/link1.dae"/>
@@ -39,5 +41,5 @@
     <link name="link2" >
       <visual>
-        <origin rpy="-1.57 0 3.14" xyz="0 0 0"/>
+        <origin rpy="-${pi/2} 0 ${pi}" xyz="0 0 0"/>
         <geometry>
           <mesh filename="file://$(find robot_bringup)/robot_mesh/link2.dae"/>
@@ -45,5 +47,5 @@
       </visual>
       <collision>
-        <origin rpy="-1.57 0 3.14" xyz="0 0 0"/>
+        <origin rpy="-${pi/2} 0 ${pi}" xyz="0 0 0"/>
         <geometry>
           <mesh filename="file://$(find robot_bringup)/robot_mesh/link2.dae"/>
@@ -57,5 +59,5 @@
     <link name="link3" >
       <visual>
-        <origin rpy="1.57 0 3.14" xyz="0 0 0"/>
+        <origin rpy="${pi/2} 0 ${pi}" xyz="0 0 0"/>
         <geometry>
           <mesh filename="file://$(find robot_bringup)/robot_mesh/link3.dae"/>
@@ -63,5 +65,5 @@
       </visual>
       <collision>
-        <origin rpy="1.57 0 3.14" xyz="0 0 0"/>
+        <origin rpy="${pi/2} 0 ${pi}" xyz="0 0 0"/>
         <geometry>
           <mesh filename="file://$(find robot_bringup)/robot_mesh/link3.dae"/>
@@ -81,5 +83,5 @@
     <link name="link4" >
       <visual>
-        <origin rpy="3.14 1.57 0" xyz="0 0 0"/>
+        <origin rpy="${pi} ${pi/2} 0" xyz="0 0 0"/>
         <geometry>
           <mesh filename="file://$(find robot_bringup)/robot_mesh/link4.dae"/>
@@ -87,5 +89,5 @@
       </visual>
       <collision>
-        <origin rpy="3.14 1.57 0" xyz="0 0 0"/>
+        <origin rpy="${pi} ${pi/2} 0" xyz="0 0 0"/>
         <geometry>
           <mesh filename="file://$(find robot_bringup)/robot_mesh/link4.dae"/>
@@ -105,5 +107,5 @@
     <link name="link4_1" >
       <visual>
-        <origin rpy="3.14 1.57 0.261" xyz="0 0 0"/>
+        <origin rpy="${pi} ${pi/2} 0.261" xyz="0 0 0"/>
         <geometry>
           <mesh filename="file://$(find robot_bringup)/robot_mesh/link4_1.dae"/>
@@ -111,5 +113,5 @@
       </visual>
       <collision>
-        <origin rpy="3.14 1.57 0.261" xyz="0 0 0"/>
+        <origin rpy="${pi} ${pi/2} 0.261" xyz="0 0 0"/>
         <geometry>
           <mesh filename="file://$(find robot_bringup)/robot_mesh/link4_1.dae"/>
@@ -123,5 +125,5 @@
     <link name="link4_2" >
       <visual>
-        <origin rpy="3.14 1.57 1.57" xyz="0 0 0"/>
+        <origin rpy="${pi} ${pi/2} ${pi/2}" xyz="0 0 0"/>
         <geometry>
           <mesh filename="file://$(find robot_bringup)/robot_mesh/link4_2.dae"/>
@@ -129,5 +131,5 @@
       </visual>
       <collision>
-        <origin rpy="3.14 1.57 1.57" xyz="0 0 0"/>
+        <origin rpy="${pi} ${pi/2} ${pi/2}" xyz="0 0 0"/>
         <geometry>
           <mesh filename="file://$(find robot_bringup)/robot_mesh/link4_2.dae"/>
@@ -174,5 +176,5 @@
       <child link="link2"/>
       <axis xyz="0 0 1" />
-      <origin xyz="0.247 0.16802 0.332" rpy="1.57 0 0" />
+      <origin xyz="0.247 0.16802 0.332" rpy="${pi/2} 0 0" />
     </joint>
     <joint name="joint3" type="continuous">
@@ -200,5 +202,5 @@
       <child link="link5"/>
       <axis xyz="0 0 1" />
-      <origin xyz="0.17227 -0.18953 0" rpy="1.57 0 0" />
+      <origin xyz="0.17227 -0.18953 0" rpy="${pi/2} 0 0" />
     </joint>
     <joint name="joint4_1" type="continuous">
@@ -207,5 +209,5 @@
       <child link="link4_1"/>
       <axis xyz="0 0 1" />
-      <origin xyz="-0.08421 0.06192 0.37687" rpy="-1.57 0.02 0" />
+      <origin xyz="-0.08421 0.06192 0.37687" rpy="-${pi/2} 0.02 0" />
     </joint>
     <joint name="joint4_2" type="continuous">

Commit message: trying to make it work with gazebo

File: robot_bringup/urdf/robot.urdf.xacro (robot description, xacro)
@@ -1,5 +1,25 @@
 <?xml version="1.0"?>
 <robot xmlns:xacro="http://www.ros.org/wiki/xacro" name="robot">
+  <xacro:macro name="mimic_joint_plugin_gazebo" params="name_prefix parent_joint mimic_joint has_pid:=false multiplier:=1.0 offset:=0 sensitiveness:=0.0 max_effort:=1.0 robot_namespace:=''">
+    <gazebo>
+      <plugin name="${name_prefix}mimic_joint_plugin" filename="libroboticsgroup_upatras_gazebo_mimic_joint_plugin.so">
+        <joint>${parent_joint}</joint>
+        <mimicJoint>${mimic_joint}</mimicJoint>
+        <xacro:if value="${has_pid}">                     <!-- if set to true, PID parameters from "/gazebo_ros_control/pid_gains/${mimic_joint}" are loaded -->
+          <hasPID />
+        </xacro:if>
+        <multiplier>${multiplier}</multiplier>
+        <offset>${offset}</offset>
+        <sensitiveness>${sensitiveness}</sensitiveness>   <!-- if absolute difference between setpoint and process value is below this threshold, do nothing; 0.0 = disable [rad] -->
+        <maxEffort>${max_effort}</maxEffort>              <!-- only taken into account if has_pid:=true [Nm] -->
+        <xacro:unless value="${robot_namespace == ''}">
+          <robotNamespace>${robot_namespace}</robotNamespace>
+        </xacro:unless>
+      </plugin>
+    </gazebo>
+  </xacro:macro>
     <!-- <xacro:property name="pi" value="3.14" /> -->
+    <link name="dummy_link" >
+    </link >
     <link name="base_link" >
         <visual>
@@ -12,12 +32,21 @@
             <origin rpy="${pi/2} 0 0" xyz="0 0 0"/>
             <geometry>
-              <mesh filename="file://$(find robot_bringup)/robot_mesh/base_link.dae"/>
+              <!-- <mesh filename="file://$(find robot_bringup)/robot_mesh/base_link.dae"/>  -->
+              <box size="0.3 0.3 0.3"/>
             </geometry>
           </collision>
           <inertial>
-            <origin xyz="0.15 0.15 .2" rpy="0 0 0"/>
-            <mass value="10000"/>
-            <inertia ixx="0" ixy="0" ixz="0" iyy="0" iyz="0" izz="0"/>
+            <mass value="50000"/>
+            <inertia ixx="0.4" ixy="0.0" ixz="0.0" iyy="0.4" iyz="0.0" izz="0.2"/>
           </inertial>
+          <surface>
+            <friction>
+              <ode>
+                <mu>100000.0</mu>
+                <mu2>100000.0</mu2>
+              </ode>
+            </friction>
+            </surface>
+            <selfCollide>false</selfCollide>
     </link >
     <link name="link1">
@@ -28,14 +57,15 @@
         </geometry>
       </visual>
-      <collision>
+      <!-- <collision>
         <origin rpy="${pi/2} 0 ${pi/2}" xyz="0 0 0"/>
         <geometry>
           <mesh filename="file://$(find robot_bringup)/robot_mesh/link1.dae"/>
         </geometry>
-      </collision>
-      <inertial>
-        <mass value="1000"/>
-        <inertia ixx="0.4" ixy="0.0" ixz="0.0" iyy="0.4" iyz="0.0" izz="0.2"/>
-      </inertial>
+      </collision> -->
+      <inertial>
+        <mass value="1000"/>
+        <inertia ixx="0.4" ixy="0.0" ixz="0.0" iyy="0.4" iyz="0.0" izz="0.2"/>
+      </inertial>
+      <selfCollide>false</selfCollide>
     </link >
     <link name="link2" >
@@ -46,14 +76,15 @@
         </geometry>
       </visual>
-      <collision>
+      <!-- <collision>
         <origin rpy="-${pi/2} 0 ${pi}" xyz="0 0 0"/>
         <geometry>
           <mesh filename="file://$(find robot_bringup)/robot_mesh/link2.dae"/>
         </geometry>
-      </collision>
-      <inertial>
-        <mass value="1000"/>
-        <inertia ixx="0.4" ixy="0.0" ixz="0.0" iyy="0.4" iyz="0.0" izz="0.2"/>
-      </inertial>
+      </collision> -->
+      <inertial>
+        <mass value="1000"/>
+        <inertia ixx="0.4" ixy="0.0" ixz="0.0" iyy="0.4" iyz="0.0" izz="0.2"/>
+      </inertial>
+      <selfCollide>false</selfCollide>
     </link >
     <link name="link3" >
@@ -64,20 +95,22 @@
         </geometry>
       </visual>
-      <collision>
+      <!-- <collision>
         <origin rpy="${pi/2} 0 ${pi}" xyz="0 0 0"/>
         <geometry>
           <mesh filename="file://$(find robot_bringup)/robot_mesh/link3.dae"/>
         </geometry>
-      </collision>
-      <inertial>
-        <mass value="1000"/>
-        <inertia ixx="0.4" ixy="0.0" ixz="0.0" iyy="0.4" iyz="0.0" izz="0.2"/>
-      </inertial>
+      </collision> -->
+      <inertial>
+        <mass value="1000"/>
+        <inertia ixx="0.4" ixy="0.0" ixz="0.0" iyy="0.4" iyz="0.0" izz="0.2"/>
+      </inertial>
+      <selfCollide>false</selfCollide>
     </link >
     <link name="link4_artificial" >
       <inertial>
         <mass value="10"/>
-        <inertia ixx="0.4" ixy="0.0" ixz="0.0" iyy="0.4" iyz="0.0" izz="0.2"/>
-      </inertial>
+        <inertia ixx="0.0004" ixy="0.0" ixz="0.0" iyy="0.0004" iyz="0.0" izz="0.0002"/>
+      </inertial>
+      <selfCollide>false</selfCollide>
     </link >
     <link name="link4" >
@@ -88,22 +121,24 @@
         </geometry>
       </visual>
-      <collision>
+      <!-- <collision>
         <origin rpy="${pi} ${pi/2} 0" xyz="0 0 0"/>
         <geometry>
           <mesh filename="file://$(find robot_bringup)/robot_mesh/link4.dae"/>
         </geometry>
-      </collision>
-      <inertial>
-        <mass value="1000"/>
-        <inertia ixx="0.4" ixy="0.0" ixz="0.0" iyy="0.4" iyz="0.0" izz="0.2"/>
-      </inertial>
+      </collision> -->
+      <inertial>
+        <mass value="1000"/>
+        <inertia ixx="0.4" ixy="0.0" ixz="0.0" iyy="0.4" iyz="0.0" izz="0.2"/>
+      </inertial>
+      <selfCollide>false</selfCollide>
     </link >
     <link name="link5" >
       <inertial>
         <mass value="10"/>
-        <inertia ixx="0.4" ixy="0.0" ixz="0.0" iyy="0.4" iyz="0.0" izz="0.2"/>
-      </inertial>
-    </link >
-    <link name="link4_1" >
+        <inertia ixx="0.004" ixy="0.0" ixz="0.0" iyy="0.004" iyz="0.0" izz="0.002"/>
+      </inertial>
+      <selfCollide>false</selfCollide>
+    </link >
+    <!-- <link name="link4_1" >
       <visual>
         <origin rpy="${pi} ${pi/2} 0.261" xyz="0 0 0"/>
@@ -165,20 +200,29 @@
       </inertial>
     </link >
+   -->
     <!-- Joints Declaration -->
-    <joint name="joint1" type="continuous">
+    <joint name="dummy_joint" type="fixed">
+      <parent link="dummy_link"/>
+      <child link="base_link"/>
+      <origin xyz="0 0 0" rpy="0 0 0" />
+    </joint>
+    <joint name="joint1" type="revolute">
       <parent link="base_link"/>
       <child link="link1"/>
+      <limit effort="100.0" lower="${-175*pi/180}" upper="${175*pi/180}" velocity="${60*pi/180}"/>
       <axis xyz="0 0 1" />
       <origin xyz="0 0 0.2645" rpy="0 0 0" />
     </joint>
-    <joint name="joint2" type="continuous">
+    <joint name="joint2" type="revolute">
       <parent link="link1"/>
       <child link="link2"/>
-      <axis xyz="0 0 1" />
-      <origin xyz="0.247 0.16802 0.332" rpy="${pi/2} 0 0" />
-    </joint>
-    <joint name="joint3" type="continuous">
+      <limit effort="100.0" lower="${-25*pi/180}" upper="${80*pi/180}" velocity="${148*pi/180}"/>
+      <axis xyz="0 0 1" />
+      <origin xyz="0.21938 0.1675 0.332" rpy="${pi/2} 0 0" />
+    </joint>
+    <joint name="joint3" type="revolute">
       <parent link="link2"/>
       <child link="link3"/>
+      <limit effort="100.0" lower="${-25*pi/180}" upper="${80*pi/180}" velocity="${148*pi/180}"/>
       <axis xyz="0 0 1" />
       <origin xyz="0 1.100 0" rpy="0 0 0" />
@@ -189,6 +233,9 @@
       <child link="link4_artificial"/>
       <axis xyz="0 0 1" />
-      <origin xyz="0.97283 0 0.1025" rpy="0 0 0" />
-    </joint>
+      <origin xyz="0.97509 0 0.1025" rpy="0 0 0" />
+    </joint>
+    <xacro:mimic_joint_plugin_gazebo name_prefix="joint4_artificial"
+    parent_joint="joint2" mimic_joint="joint4_artificial"
+    has_pid="false" multiplier="-1.0" max_effort="10.0" />
     <joint name="joint4" type="continuous">
       <mimic joint="joint3" multiplier="-1" offset="0" />
@@ -198,11 +245,15 @@
       <origin xyz="0 0 0" rpy="0 0 0" />
     </joint>
-    <joint name="joint5" type="continuous">
+    <xacro:mimic_joint_plugin_gazebo name_prefix="joint4"
+    parent_joint="joint3" mimic_joint="joint4"
+    has_pid="false" multiplier="-1.0" max_effort="10.0" />
+    <joint name="joint5" type="revolute">
       <parent link="link4"/>
       <child link="link5"/>
       <axis xyz="0 0 1" />
-      <origin xyz="0.17227 -0.18953 0" rpy="${pi/2} 0 0" />
-    </joint>
-    <joint name="joint4_1" type="continuous">
+      <limit effort="1000.0" lower="${-360*pi/180}" upper="${360*pi/180}" velocity="${148*pi/180}"/>
+      <origin xyz="0.1718 -0.18957 0" rpy="${pi/2} 0 0" />
+    </joint>
+    <!-- <joint name="joint4_1" type="continuous">
       <mimic joint="joint2" multiplier="-1" offset="0" />
       <parent link="link1"/>
@@ -231,5 +282,5 @@
       <axis xyz="0 0 1" />
       <origin xyz="0 0 0" rpy="0 0 0" />
-    </joint>
+    </joint> -->
     <!-- Transmission -->
     <gazebo>
@@ -241,5 +292,5 @@
     <transmission name="tran1">
       <type>transmission_interface/SimpleTransmission</type>
-      <actuator name="$base_link_motor">
+      <actuator name="motor1">
         <mechanicalReduction>1</mechanicalReduction>
         <hardwareInterface>hardware_interface/EffortJointInterface</hardwareInterface>
@@ -251,5 +302,5 @@
     <transmission name="tran2">
       <type>transmission_interface/SimpleTransmission</type>
-      <actuator name="$link2_motor">
+      <actuator name="motor2">
         <mechanicalReduction>1</mechanicalReduction>
         <hardwareInterface>hardware_interface/EffortJointInterface</hardwareInterface>
@@ -261,9 +312,19 @@
     <transmission name="tran3">
       <type>transmission_interface/SimpleTransmission</type>
-      <actuator name="$link3_motor">
+      <actuator name="motor3">
         <mechanicalReduction>1</mechanicalReduction>
         <hardwareInterface>hardware_interface/EffortJointInterface</hardwareInterface>
       </actuator>
       <joint name="joint3">
+        <hardwareInterface>hardware_interface/EffortJointInterface</hardwareInterface>
+      </joint>
+    </transmission>
+    <transmission name="tran4">
+      <type>transmission_interface/SimpleTransmission</type>
+      <actuator name="motor5">
+        <mechanicalReduction>1</mechanicalReduction>
+        <hardwareInterface>hardware_interface/EffortJointInterface</hardwareInterface>
+      </actuator>
+      <joint name="joint5">
         <hardwareInterface>hardware_interface/EffortJointInterface</hardwareInterface>
       </joint>

Commit message: updated readme

File: robot_bringup/urdf/robot.urdf.xacro (robot description, xacro)
@@ -19,5 +19,5 @@
     </gazebo>
   </xacro:macro>
-    <!-- <xacro:property name="pi" value="3.14" /> -->
+    <xacro:property name="path" value="model://" />
     <link name="dummy_link" >
     </link >

Commit message: managed to pick up a can in gazebo

File: robot_bringup/urdf/robot.urdf.xacro (robot description, xacro)
@@ -138,4 +138,80 @@
       <selfCollide>false</selfCollide>
     </link >
+    <link name="link6_1" >
+      <visual>
+        <origin rpy="${pi} ${pi/2} 0" xyz="0.1 0 0"/>
+        <geometry>
+          <cylinder radius="0.02" length="0.2"/>
+        </geometry>
+      </visual>
+      <collision>
+        <origin rpy="${pi} ${pi/2} 0" xyz="0.1 0 0"/>
+        <geometry>
+          <cylinder radius="0.02" length="0.2"/>
+        </geometry>
+      </collision>
+      <inertial>
+        <mass value="1"/>
+        <inertia ixx="0.001" ixy="0.0" ixz="0.0" iyy="0.001" iyz="0.0" izz="0.001"/>
+      </inertial>
+      <surface>
+        <friction>
+          <ode>
+            <mu>1</mu>
+            <mu2>1</mu2>
+          </ode>
+          <torsional>
+            <ode/>
+          </torsional>
+        </friction>
+        <contact>
+          <ode>
+            <kp>1e+07</kp>
+            <kd>1</kd>
+            <min_depth>0.001</min_depth>
+            <max_vel>0.1</max_vel>
+          </ode>
+        </contact>
+        <bounce/>
+      </surface>
+    </link >
+    <link name="link6_2" >
+      <visual>
+        <origin rpy="${pi} ${pi/2} 0" xyz="0.1 0 0"/>
+        <geometry>
+          <cylinder radius="0.02" length="0.2"/>
+        </geometry>
+      </visual>
+      <collision>
+        <origin rpy="${pi} ${pi/2} 0" xyz="0.1 0 0"/>
+        <geometry>
+          <cylinder radius="0.02" length="0.2"/>
+        </geometry>
+      </collision>
+      <inertial>
+        <mass value="1"/>
+        <inertia ixx="0.001" ixy="0.0" ixz="0.0" iyy="0.001" iyz="0.0" izz="0.001"/>
+      </inertial>
+      <surface>
+        <friction>
+          <ode>
+            <mu>1</mu>
+            <mu2>1</mu2>
+          </ode>
+          <torsional>
+            <ode/>
+          </torsional>
+        </friction>
+        <contact>
+          <ode>
+            <kp>1e+07</kp>
+            <kd>1</kd>
+            <min_depth>0.001</min_depth>
+            <max_vel>0.1</max_vel>
+          </ode>
+        </contact>
+        <bounce/>
+      </surface>
+    </link >
     <!-- <link name="link4_1" >
       <visual>
@@ -257,4 +333,24 @@
       <dynamics damping="0.5" friction="0.0"/>
     </joint>
+    <joint name="joint6_1" type="prismatic">
+      <parent link="link5"/>
+      <child link="link6_1"/>
+      <axis xyz="0 1 0" />
+      <limit effort="100.0" lower="-0.05" upper="0.15" velocity="${148*pi/180}"/>
+      <origin xyz="0 0.05 0.1" rpy="0 0 0" />
+      <dynamics damping="0.5" friction="5.0"/>
+    </joint>
+    <joint name="joint6_2" type="prismatic">
+      <mimic joint="joint6_1" multiplier="-1" offset="0" />
+      <parent link="link5"/>
+      <child link="link6_2"/>
+      <axis xyz="0 1 0" />
+      <limit effort="100.0" lower="-0.05" upper="0.15" velocity="${148*pi/180}"/>
+      <origin xyz="0 -0.05 0.1" rpy="0 0 0" />
+      <dynamics damping="0.5" friction="5.0"/>
+    </joint>
+    <xacro:mimic_joint_plugin_gazebo name_prefix="joint4"
+    parent_joint="joint6_1" mimic_joint="joint6_2"
+    has_pid="false" multiplier="-1.0" max_effort="100.0" />
     <!-- <joint name="joint4_1" type="continuous">
       <mimic joint="joint2" multiplier="-1" offset="0" />
@@ -344,3 +440,13 @@
       </joint>
     </transmission>
+    <transmission name="tran5">
+      <type>transmission_interface/SimpleTransmission</type>
+      <actuator name="motor6">
+        <mechanicalReduction>1</mechanicalReduction>
+        <hardwareInterface>hardware_interface/PositionJointInterface</hardwareInterface>
+      </actuator>
+      <joint name="joint6_1">
+        <hardwareInterface>hardware_interface/PositionJointInterface</hardwareInterface>
+      </joint>
+    </transmission>
   </robot>

File: robot_bringup/urdf/robot_rviz.urdf.xacro (robot description, xacro)
@@ -19,5 +19,5 @@
     </gazebo>
   </xacro:macro>
-   <xacro:property name="path" value="/media/andre/Andre/robot_mesh" />
+  <xacro:property name="path" value="~/../../media/andre/Andre/robot_mesh" />
     <!-- <xacro:property name="pi" value="3.14" /> -->
     <link name="dummy_link" >
@@ -27,5 +27,5 @@
             <origin rpy="${pi/2} 0 0" xyz="0 0 0"/>
             <geometry>
-              <mesh filename="${path}/base_link.dae"/>
+              <mesh filename="~/../../media/andre/Andre/robot_mesh/base_link.dae"/>
             </geometry>
           </visual>
@@ -141,4 +141,42 @@
       <selfCollide>false</selfCollide>
     </link >
+    <link name="link6_1" >
+      <visual>
+        <origin rpy="${pi} ${pi/2} 0" xyz="0.1 0 0"/>
+        <geometry>
+          <cylinder radius="0.02" length="0.2"/>
+        </geometry>
+      </visual>
+      <collision>
+        <origin rpy="${pi} ${pi/2} 0" xyz="0.1 0 0"/>
+        <geometry>
+          <cylinder radius="0.02" length="0.2"/>
+        </geometry>
+      </collision>
+      <inertial>
+        <mass value="1"/>
+        <inertia ixx="0.001" ixy="0.0" ixz="0.0" iyy="0.001" iyz="0.0" izz="0.001"/>
+      </inertial>
+      <selfCollide>false</selfCollide>
+    </link >
+    <link name="link6_2" >
+      <visual>
+        <origin rpy="${pi} ${pi/2} 0" xyz="0.1 0 0"/>
+        <geometry>
+          <cylinder radius="0.02" length="0.2"/>
+        </geometry>
+      </visual>
+      <collision>
+        <origin rpy="${pi} ${pi/2} 0" xyz="0.1 0 0"/>
+        <geometry>
+          <cylinder radius="0.02" length="0.2"/>
+        </geometry>
+      </collision>
+      <inertial>
+        <mass value="1"/>
+        <inertia ixx="0.001" ixy="0.0" ixz="0.0" iyy="0.001" iyz="0.0" izz="0.001"/>
+      </inertial>
+      <selfCollide>false</selfCollide>
+    </link >
     <link name="link4_1" >
       <visual>
@@ -255,4 +293,24 @@
       <origin xyz="0.1718 -0.18957 0" rpy="${pi/2} 0 0" />
     </joint>
+    <joint name="joint6_1" type="prismatic">
+      <parent link="link5"/>
+      <child link="link6_1"/>
+      <axis xyz="0 1 0" />
+      <limit effort="10.0" lower="-0.05" upper="0.15" velocity="${148*pi/180}"/>
+      <origin xyz="0 0.05 0.1" rpy="0 0 0" />
+      <dynamics damping="0.5" friction="0.0"/>
+    </joint>
+    <joint name="joint6_2" type="prismatic">
+      <mimic joint="joint6_1" multiplier="-1" offset="0" />
+      <parent link="link5"/>
+      <child link="link6_2"/>
+      <axis xyz="0 1 0" />
+      <limit effort="10.0" lower="-0.05" upper="0.15" velocity="${148*pi/180}"/>
+      <origin xyz="0 -0.05 0.1" rpy="0 0 0" />
+      <dynamics damping="0.5" friction="0.0"/>
+    </joint>
+    <xacro:mimic_joint_plugin_gazebo name_prefix="joint4"
+    parent_joint="joint6_1" mimic_joint="joint6_2"
+    has_pid="false" multiplier="-1.0" max_effort="10.0" />
     <joint name="joint4_1" type="continuous">
       <mimic joint="joint2" multiplier="-1" offset="0" />
