Commit message: cleaned code

File: robot_bringup/urdf/robot.urdf.xacro (robot description, xacro)
@@ -291,5 +291,5 @@
       <parent link="link1"/>
       <child link="link2"/>
-      <limit effort="1000000.0" lower="${-25*pi/180}" upper="${80*pi/180}" velocity="${148*pi/180}"/>
+      <limit effort="1000000.0" lower="${-80*pi/180}" upper="${25*pi/180}" velocity="${148*pi/180}"/>
       <axis xyz="0 0 1" />
       <origin xyz="0.21938 0.1675 0.332" rpy="${pi/2} 0 0" />
@@ -299,5 +299,5 @@
       <parent link="link2"/>
       <child link="link3"/>
-      <limit effort="1000000.0" lower="${-25*pi/180}" upper="${80*pi/180}" velocity="${148*pi/180}"/>
+      <limit effort="1000000.0" lower="${-80*pi/180}" upper="${25*pi/180}" velocity="${148*pi/180}"/>
       <axis xyz="0 0 1" />
       <origin xyz="0 1.100 0" rpy="0 0 0" />

File: robot_bringup/urdf/robot_rviz.urdf.xacro (robot description, xacro)
@@ -145,5 +145,6 @@
         <origin rpy="${pi} ${pi/2} 0" xyz="0.1 0 0"/>
         <geometry>
-          <cylinder radius="0.02" length="0.2"/>
+          <!-- <cylinder radius="0.02" length="0.2"/> -->
+          <box size="0.05 0.02 0.2" />
         </geometry>
       </visual>
@@ -151,5 +152,5 @@
         <origin rpy="${pi} ${pi/2} 0" xyz="0.1 0 0"/>
         <geometry>
-          <cylinder radius="0.02" length="0.2"/>
+          <box size="0.05 0.02 0.2" />
         </geometry>
       </collision>
@@ -164,5 +165,5 @@
         <origin rpy="${pi} ${pi/2} 0" xyz="0.1 0 0"/>
         <geometry>
-          <cylinder radius="0.02" length="0.2"/>
+          <box size="0.05 0.02 0.2" />
         </geometry>
       </visual>
@@ -170,5 +171,5 @@
         <origin rpy="${pi} ${pi/2} 0" xyz="0.1 0 0"/>
         <geometry>
-          <cylinder radius="0.02" length="0.2"/>
+          <box size="0.05 0.02 0.2" />
         </geometry>
       </collision>
@@ -255,14 +256,16 @@
       <parent link="link1"/>
       <child link="link2"/>
-      <limit effort="100.0" lower="${-25*pi/180}" upper="${80*pi/180}" velocity="${148*pi/180}"/>
+      <limit effort="1000000.0" lower="${-80*pi/180}" upper="${25*pi/180}" velocity="${148*pi/180}"/>
       <axis xyz="0 0 1" />
       <origin xyz="0.21938 0.1675 0.332" rpy="${pi/2} 0 0" />
+      <dynamics damping="0.5" friction="0.0"/>
     </joint>
     <joint name="joint3" type="revolute">
       <parent link="link2"/>
       <child link="link3"/>
-      <limit effort="100.0" lower="${-25*pi/180}" upper="${80*pi/180}" velocity="${148*pi/180}"/>
+      <limit effort="1000000.0" lower="${-80*pi/180}" upper="${25*pi/180}" velocity="${148*pi/180}"/>
       <axis xyz="0 0 1" />
       <origin xyz="0 1.100 0" rpy="0 0 0" />
+      <dynamics damping="0.5" friction="0.0"/>
     </joint>
     <joint name="joint4_artificial" type="continuous">

Commit message: changed tool to box

File: robot_bringup/urdf/robot.urdf.xacro (robot description, xacro)
@@ -142,5 +142,5 @@
         <origin rpy="${pi} ${pi/2} 0" xyz="0.1 0 0"/>
         <geometry>
-          <cylinder radius="0.02" length="0.2"/>
+          <box size="0.05 0.02 0.2" />
         </geometry>
       </visual>
@@ -148,5 +148,5 @@
         <origin rpy="${pi} ${pi/2} 0" xyz="0.1 0 0"/>
         <geometry>
-          <cylinder radius="0.02" length="0.2"/>
+          <box size="0.05 0.02 0.2" />
         </geometry>
       </collision>
@@ -180,5 +180,5 @@
         <origin rpy="${pi} ${pi/2} 0" xyz="0.1 0 0"/>
         <geometry>
-          <cylinder radius="0.02" length="0.2"/>
+          <box size="0.05 0.02 0.2" />
         </geometry>
       </visual>
@@ -186,5 +186,5 @@
         <origin rpy="${pi} ${pi/2} 0" xyz="0.1 0 0"/>
         <geometry>
-          <cylinder radius="0.02" length="0.2"/>
+          <box size="0.05 0.02 0.2" />
         </geometry>
       </collision>
@@ -350,7 +350,7 @@
       <dynamics damping="0.5" friction="5.0"/>
     </joint>
-    <xacro:mimic_joint_plugin_gazebo name_prefix="joint4"
+    <xacro:mimic_joint_plugin_gazebo name_prefix="joint6_1"
     parent_joint="joint6_1" mimic_joint="joint6_2"
-    has_pid="false" multiplier="-1.0" max_effort="100.0" />
+    has_pid="false" multiplier="-1.0" max_effort="10.0" />
     <!-- <joint name="joint4_1" type="continuous">
       <mimic joint="joint2" multiplier="-1" offset="0" />
